File: display/display.sch (KiCad schematic (older format))
At the start: 1 part, among them J1 Conn_01x03_Male

Commit message: WIP peer
Parts:
- removed J1: Conn_01x03_Male, display:strip_connector, symbol display:Conn_01x03_Male
- added J1: Raspberry Pi, Arduino:raspberrypi_2_3, symbol Connector_Generic:Conn_02x20_Odd_Even
- added LS0: LED Strip 0, display:strip_connector_hole, symbol Connector:Conn_01x03_Male
- added LS1: LED Strip 1, display:strip_connector_hole, symbol Connector:Conn_01x03_Male
- added LS10: LED Strip A, display:strip_connector_hole, symbol Connector:Conn_01x03_Male
- added LS11: LED Strip B, display:strip_connector_hole, symbol Connector:Conn_01x03_Male
- added LS12: LED Strip C, display:strip_connector_hole, symbol Connector:Conn_01x03_Male
- added LS13: LED Strip D, display:strip_connector_hole, symbol Connector:Conn_01x03_Male
- added LS14: LED Strip E, display:strip_connector_hole, symbol Connector:Conn_01x03_Male
- added LS15: LED Strip F, display:strip_connector_hole, symbol Connector:Conn_01x03_Male
- added LS2: LED Strip 2, display:strip_connector_hole, symbol Connector:Conn_01x03_Male
- added LS3: LED Strip 3, display:strip_connector_hole, symbol Connector:Conn_01x03_Male
- added LS4: LED Strip 4, display:strip_connector_hole, symbol Connector:Conn_01x03_Male
- added LS5: LED Strip 5, display:strip_connector_hole, symbol Connector:Conn_01x03_Male
- added LS6: LED Strip 6, display:strip_connector_hole, symbol Connector:Conn_01x03_Male
- added LS7: LED Strip 7, display:strip_connector_hole, symbol Connector:Conn_01x03_Male
- added LS8: LED Strip 8, display:strip_connector_hole, symbol Connector:Conn_01x03_Male
- added LS9: LED Strip 9, display:strip_connector_hole, symbol Connector:Conn_01x03_Male
- added XA1: Arduino_Mega2560_Shield_redux, display:Arduino_Mega2560_Shield_redux, symbol display:Arduino_Mega2560_Shield_redux
Connections:
- new net +3V3: J1.1 (Pin_1), J1.17 (Pin_17)
- new net +5V: J1.2 (Pin_2), J1.4 (Pin_4), LS0.1 (Pin_1), LS1.1 (Pin_1), LS10.1 (Pin_1), LS11.1 (Pin_1), LS12.1 (Pin_1), LS13.1 (Pin_1), LS14.1 (Pin_1), LS15.1 (Pin_1), LS2.1 (Pin_1), LS3.1 (Pin_1), LS4.1 (Pin_1), LS5.1 (Pin_1), LS6.1 (Pin_1), LS7.1 (Pin_1), LS8.1 (Pin_1), LS9.1 (Pin_1), XA1.5V1 (5V), XA1.5V3 (5V), XA1.5V4 (5V)
- new net GND: J1.14 (Pin_14), J1.20 (Pin_20), J1.25 (Pin_25), J1.30 (Pin_30), J1.34 (Pin_34), J1.39 (Pin_39), J1.6 (Pin_6), J1.9 (Pin_9), LS0.3 (Pin_3), LS1.3 (Pin_3), LS10.3 (Pin_3), LS11.3 (Pin_3), LS12.3 (Pin_3), LS13.3 (Pin_3), LS14.3 (Pin_3), LS15.3 (Pin_3), LS2.3 (Pin_3), LS3.3 (Pin_3), LS4.3 (Pin_3), LS5.3 (Pin_3), LS6.3 (Pin_3), LS7.3 (Pin_3), LS8.3 (Pin_3), LS9.3 (Pin_3), XA1.GND1 (GND), XA1.GND2 (GND), XA1.GND3 (GND), XA1.GND5 (GND), XA1.GND6 (GND)
- new net d0: LS0.2 (Pin_2), XA1.D0 (D0_RX0)
- new net d1: LS1.2 (Pin_2), XA1.D1 (D1_TX0)
- new net d2: LS2.2 (Pin_2), XA1.D2 (D2_INT0)
- new net d3: LS3.2 (Pin_2), XA1.D3 (D3_INT1)
- new net d4: LS4.2 (Pin_2), XA1.D4
- new net d5: LS5.2 (Pin_2), XA1.D5
- new net d6: LS6.2 (Pin_2), XA1.D6
- new net d7: LS7.2 (Pin_2), XA1.D7
- new net d8: LS8.2 (Pin_2), XA1.D8
- new net d9: LS9.2 (Pin_2), XA1.D9
- new net dA: LS10.2 (Pin_2), XA1.D10
- new net dB: LS11.2 (Pin_2), XA1.D11
- new net dC: LS12.2 (Pin_2), XA1.D12
- new net dD: LS13.2 (Pin_2), XA1.D13
- new net dE: LS14.2 (Pin_2), XA1.SDA
- new net dF: LS15.2 (Pin_2), XA1.SCL
