File: display/display.kicad_pcb (KiCad board)
At the start: 2 copper layers, 76.2 x 50.8 mm, 6 parts

Commit message: Connect all signals
Parts:
- added REF**: strip_connector, display:strip_connector, F.Cu at (290.0, 120.0)
- added REF**: strip_connector, display:strip_connector, F.Cu at (140.0, 120.0)
- added REF**: strip_connector, display:strip_connector, F.Cu at (123.3, 120.0)
- added REF**: strip_connector, display:strip_connector, F.Cu at (106.7, 120.0)
- added REF**: strip_connector, display:strip_connector, F.Cu at (90.0, 120.0)
- added REF**: strip_connector, display:strip_connector, F.Cu at (223.3, 120.0)
- added REF**: strip_connector, display:strip_connector, F.Cu at (256.7, 120.0)
- added REF**: strip_connector, display:strip_connector, F.Cu at (273.3, 120.0)
- added REF**: strip_connector, display:strip_connector, F.Cu at (190.0, 120.0)
- added REF**: strip_connector, display:strip_connector, F.Cu at (206.7, 120.0)
- added REF**: strip_connector, display:strip_connector, F.Cu at (173.3, 120.0)
- added REF**: strip_connector, display:strip_connector, F.Cu at (240.0, 120.0)
- added REF**: strip_connector, display:strip_connector, F.Cu at (156.7, 120.0)
- moved REF** 19.0 mm to (77.5, 66.4)
- moved REF** 19.0 mm to (48.5, 67.5)
- moved REF** 19.0 mm to (38.1, 67.3)
Routing:
- net (no net): track 493.6 -> 3764.0 mm, vias 4 -> 17
Other:
- board size 76.2 x 50.8 mm -> 279.1 x 72.1 mm

Commit message: New board dimensions
6mm spacing to left/right
9cm absolute height
Parts:
- added REF**: Pad, Connector_Wire:SolderWirePad_1x01_SMD_5x10mm, F.Cu at (298.4, 87.6)
- added REF**: Pad, Connector_Wire:SolderWirePad_1x01_SMD_5x10mm, F.Cu at (31.8, 87.6)
- GND: renamed from REF**; value SolderWirePad_1x01_SMD_5x10mm -> GND
- VCC: renamed from REF**; value SolderWirePad_1x01_SMD_5x10mm -> VCC
- moved GND 16.5 mm to (48.5, 51.0)
- moved VCC 16.5 mm to (38.1, 50.8)
- moved REF** 16.5 mm to (77.5, 49.9)
Routing:
- net (no net): track 3764.0 -> 4099.0 mm
Other:
- board size 279.1 x 72.1 mm -> 273.1 x 90 mm

Commit message: PoC arduino pins
Parts:
- removed the REF** at (77.5, 49.9)
- added RP?: Raspberry_Pi_2_3, Arduino:raspberrypi_2_3, B.Cu at (242.6, 49.5)
- added XA**: Arduino_Mega2560_Shield-moded, Arduino:Arduino_Mega2560_Shield-moded, B.Cu at (63.5, 45.7)
Routing:
- net (no net): track 4099.0 -> 3549.5 mm

Commit message: WIP peer
Parts:
- added J1: Raspberry Pi, Arduino:raspberrypi_2_3, F.Cu at (363.2, 6.35)
- added LS0: LED Strip 0, display:strip_connector_hole, F.Cu at (469.2, -23.5)
- added LS1: LED Strip 1, display:strip_connector_hole, F.Cu at (457.2, -12.3)
- added LS10: LED Strip A, display:strip_connector_hole, F.Cu at (457.2, -34.7)
- added LS11: LED Strip B, display:strip_connector_hole, F.Cu at (424.4, 20.0)
- added LS12: LED Strip C, display:strip_connector_hole, F.Cu at (445.2, -34.7)
- added LS13: LED Strip D, display:strip_connector_hole, F.Cu at (457.2, -45.9)
- added LS14: LED Strip E, display:strip_connector_hole, F.Cu at (424.4, 8.77)
- added LS15: LED Strip F, display:strip_connector_hole, F.Cu at (445.2, -45.9)
- added LS2: LED Strip 2, display:strip_connector_hole, F.Cu at (424.4, 31.2)
- added LS3: LED Strip 3, display:strip_connector_hole, F.Cu at (445.2, -12.3)
- added LS4: LED Strip 4, display:strip_connector_hole, F.Cu at (457.2, -23.5)
- added LS5: LED Strip 5, display:strip_connector_hole, F.Cu at (469.2, -34.7)
- added LS6: LED Strip 6, display:strip_connector_hole, F.Cu at (481.2, -45.9)
- added LS7: LED Strip 7, display:strip_connector_hole, F.Cu at (436.4, 8.77)
- added LS8: LED Strip 8, display:strip_connector_hole, F.Cu at (469.2, -45.9)
- added LS9: LED Strip 9, display:strip_connector_hole, F.Cu at (445.2, -23.5)
- added XA1: Arduino_Mega2560_Shield_redux, display:Arduino_Mega2560_Shield_redux, F.Cu at (337.1, 1.53)
Routing:
- net (no net): track 3549.5 -> 3551.9 mm

Commit message: Revive project
- Hopefully correct footprint for Arduino Mega
- Replaced all connectors with the one from the schematic footprint
- Replaced pi header with the one from the schematic
- Added infill (front & back) for easy grounding

We can now proceed to wire everything up, mainly the connection between
Arduino and Pi.
Parts:
- removed the REF** at (240.0, 120.0)
- removed the REF** at (156.7, 120.0)
- removed the REF** at (140.0, 120.0)
- removed the REF** at (123.3, 120.0)
- removed the REF** at (106.7, 120.0)
- removed the REF** at (90.0, 120.0)
- removed the REF** at (73.3, 120.0)
- removed the REF** at (56.7, 120.0)
- removed the REF** at (40.0, 120.0)
- removed the REF** at (290.0, 120.0)
- removed the REF** at (223.3, 120.0)
- removed the REF** at (256.7, 120.0)
- removed the REF** at (273.3, 120.0)
- removed the REF** at (190.0, 120.0)
- removed the REF** at (206.7, 120.0)
- removed the REF** at (173.3, 120.0)
- removed RP?: Raspberry_Pi_2_3, Arduino:raspberrypi_2_3
- removed XA**: Arduino_Mega2560_Shield-moded, Arduino:Arduino_Mega2560_Shield-moded
- J1: moved to B.Cu
- XA1: footprint display:Arduino_Mega2560_Shield_redux -> Arduino:Arduino_Mega2560_Shield; moved to B.Cu
- moved LS15 438.2 mm to (40.0, 120.6)
- moved LS13 418.5 mm to (73.3, 120.6)
- moved LS12 387.8 mm to (90.0, 120.6)
- moved LS14 384.4 mm to (56.7, 120.7)
- moved LS10 368.3 mm to (123.4, 120.6)
- moved LS8 354.1 mm to (156.7, 120.6)
- moved LS9 337.5 mm to (140.0, 120.6)
- moved LS6 335.5 mm to (190.0, 120.6)
- moved LS11 333.3 mm to (106.6, 120.6)
- moved LS5 305.1 mm to (206.7, 120.7)
- moved LS7 285.8 mm to (173.4, 120.7)
- moved XA1 277.1 mm to (63.5, 45.8)
- moved LS4 274.8 mm to (223.3, 120.6)
- moved LS3 244.5 mm to (240.0, 120.7)
- moved LS0 230.0 mm to (290.0, 120.6)
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Connections:
- GND pad 2: (no net) -> GND
- J1 pad 10: Net-(J1-Pad10) -> unconnected-(J1-Pad10)
- J1 pad 11: Net-(J1-Pad11) -> unconnected-(J1-Pad11)
- J1 pad 12: Net-(J1-Pad12) -> unconnected-(J1-Pad12)
- J1 pad 13: Net-(J1-Pad13) -> unconnected-(J1-Pad13)
- J1 pad 15: Net-(J1-Pad15) -> unconnected-(J1-Pad15)
- J1 pad 16: Net-(J1-Pad16) -> unconnected-(J1-Pad16)
- J1 pad 18: Net-(J1-Pad18) -> unconnected-(J1-Pad18)
- J1 pad 19: Net-(J1-Pad19) -> unconnected-(J1-Pad19)
- J1 pad 21: Net-(J1-Pad21) -> unconnected-(J1-Pad21)
- J1 pad 22: Net-(J1-Pad22) -> unconnected-(J1-Pad22)
- J1 pad 23: Net-(J1-Pad23) -> unconnected-(J1-Pad23)
- J1 pad 24: Net-(J1-Pad24) -> unconnected-(J1-Pad24)
- J1 pad 26: Net-(J1-Pad26) -> unconnected-(J1-Pad26)
- J1 pad 27: Net-(J1-Pad27) -> unconnected-(J1-Pad27)
- J1 pad 28: Net-(J1-Pad28) -> unconnected-(J1-Pad28)
- J1 pad 29: Net-(J1-Pad29) -> unconnected-(J1-Pad29)
- J1 pad 3: Net-(J1-Pad3) -> unconnected-(J1-Pad3)
- J1 pad 31: Net-(J1-Pad31) -> unconnected-(J1-Pad31)
- J1 pad 32: Net-(J1-Pad32) -> unconnected-(J1-Pad32)
- J1 pad 33: Net-(J1-Pad33) -> unconnected-(J1-Pad33)
- J1 pad 35: Net-(J1-Pad35) -> unconnected-(J1-Pad35)
- J1 pad 36: Net-(J1-Pad36) -> unconnected-(J1-Pad36)
- J1 pad 37: Net-(J1-Pad37) -> unconnected-(J1-Pad37)
- J1 pad 38: Net-(J1-Pad38) -> unconnected-(J1-Pad38)
- J1 pad 40: Net-(J1-Pad40) -> unconnected-(J1-Pad40)
- J1 pad 5: Net-(J1-Pad5) -> unconnected-(J1-Pad5)
- J1 pad 7: Net-(J1-Pad7) -> unconnected-(J1-Pad7)
- J1 pad 8: Net-(J1-Pad8) -> unconnected-(J1-Pad8)
- VCC pad 1: (no net) -> +5V
- XA1 pad 3V3: Net-(XA1-Pad3V3) -> unconnected-(XA1-Pad3V3)
- XA1 pad 5V1: +5V -> unconnected-(XA1-Pad5V1)
- XA1 pad A0: Net-(XA1-PadA0) -> unconnected-(XA1-PadA0)
- XA1 pad A1: Net-(XA1-PadA1) -> unconnected-(XA1-PadA1)
- XA1 pad A10: Net-(XA1-PadA10) -> unconnected-(XA1-PadA10)
- XA1 pad A11: Net-(XA1-PadA11) -> unconnected-(XA1-PadA11)
- XA1 pad A12: Net-(XA1-PadA12) -> unconnected-(XA1-PadA12)
- XA1 pad A13: Net-(XA1-PadA13) -> unconnected-(XA1-PadA13)
- XA1 pad A14: Net-(XA1-PadA14) -> unconnected-(XA1-PadA14)
- XA1 pad A15: Net-(XA1-PadA15) -> unconnected-(XA1-PadA15)
- XA1 pad A2: Net-(XA1-PadA2) -> unconnected-(XA1-PadA2)
- XA1 pad A3: Net-(XA1-PadA3) -> unconnected-(XA1-PadA3)
- XA1 pad A4: Net-(XA1-PadA4) -> unconnected-(XA1-PadA4)
- XA1 pad A5: Net-(XA1-PadA5) -> unconnected-(XA1-PadA5)
- XA1 pad A6: Net-(XA1-PadA6) -> unconnected-(XA1-PadA6)
- XA1 pad A7: Net-(XA1-PadA7) -> unconnected-(XA1-PadA7)
- XA1 pad A8: Net-(XA1-PadA8) -> unconnected-(XA1-PadA8)
- XA1 pad A9: Net-(XA1-PadA9) -> unconnected-(XA1-PadA9)
- XA1 pad AREF: Net-(XA1-PadAREF) -> unconnected-(XA1-PadAREF)
- XA1 pad D14: Net-(XA1-PadD14) -> unconnected-(XA1-PadD14)
- XA1 pad D15: Net-(XA1-PadD15) -> unconnected-(XA1-PadD15)
- XA1 pad D16: Net-(XA1-PadD16) -> unconnected-(XA1-PadD16)
- XA1 pad D17: Net-(XA1-PadD17) -> unconnected-(XA1-PadD17)
- XA1 pad D18: Net-(XA1-PadD18) -> unconnected-(XA1-PadD18)
- XA1 pad D19: Net-(XA1-PadD19) -> unconnected-(XA1-PadD19)
- XA1 pad D20: Net-(XA1-PadD20) -> unconnected-(XA1-PadD20)
- XA1 pad D21: Net-(XA1-PadD21) -> unconnected-(XA1-PadD21)
- XA1 pad D22: Net-(XA1-PadD22) -> /dE
- XA1 pad D23: Net-(XA1-PadD23) -> /dF
- XA1 pad D24: Net-(XA1-PadD24) -> unconnected-(XA1-PadD24)
- XA1 pad D25: Net-(XA1-PadD25) -> unconnected-(XA1-PadD25)
- XA1 pad D46: Net-(XA1-PadD46) -> unconnected-(XA1-PadD46)
- XA1 pad D47: Net-(XA1-PadD47) -> unconnected-(XA1-PadD47)
- XA1 pad D48: Net-(XA1-PadD48) -> unconnected-(XA1-PadD48)
- XA1 pad D49: Net-(XA1-PadD49) -> unconnected-(XA1-PadD49)
- XA1 pad D50: Net-(XA1-PadD50) -> unconnected-(XA1-PadD50)
- XA1 pad D51: Net-(XA1-PadD51) -> unconnected-(XA1-PadD51)
- XA1 pad D52: Net-(XA1-PadD52) -> unconnected-(XA1-PadD52)
- XA1 pad D53: Net-(XA1-PadD53) -> unconnected-(XA1-PadD53)
- XA1 pad GND1: GND -> unconnected-(XA1-PadGND1)
- XA1 pad IORF: Net-(XA1-PadIORF) -> unconnected-(XA1-PadIORF)
- XA1 pad RST1: Net-(XA1-PadRST1) -> unconnected-(XA1-PadRST1)
- XA1 pad SCL: /dF -> unconnected-(XA1-PadSCL)
- XA1 pad SDA: /dE -> unconnected-(XA1-PadSDA)
- XA1 pad VIN: Net-(XA1-PadVIN) -> unconnected-(XA1-PadVIN)
Routing:
- net (no net): track 3551.9 -> 2.41 mm, vias 17 -> 0
- net +5V: track 0.00 -> 734.0 mm
- net /d0: track 0.00 -> 201.2 mm
- net /d1: track 0.00 -> 193.1 mm
- net /d2: track 0.00 -> 187.0 mm
- net /d3: track 0.00 -> 173.8 mm
- net /d4: track 0.00 -> 160.7 mm
- net /d5: track 0.00 -> 146.0 mm
- net /d6: track 0.00 -> 127.2 mm
- net /d7: track 0.00 -> 107.0 mm
- net /d8: track 0.00 -> 106.8 mm
- net /d9: track 0.00 -> 89.2 mm
- net unconnected-(XA1-PadSCL): track 0.00 -> 80.0 mm
- net /dA: track 0.00 -> 76.4 mm
- net unconnected-(XA1-PadSDA): track 0.00 -> 65.1 mm
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- added copper zone on B.Cu, net GND
- added copper zone on F.Cu, net GND
Other:
- net class Default removed

Commit message: Update to kicad 8
Connections:
- XA1 pad D22: /dE -> unconnected-(XA1-PadD22)
- XA1 pad D23: /dF -> unconnected-(XA1-PadD23)
- XA1 pad SCL: unconnected-(XA1-PadSCL) -> /dF
- XA1 pad SDA: unconnected-(XA1-PadSDA) -> /dE
Routing:
- net unconnected-(XA1-PadSCL): track 80.0 -> 0.00 mm
- net /dF: track 0.00 -> 80.0 mm
- net unconnected-(XA1-PadSDA): track 65.1 -> 0.00 mm
- net /dE: track 0.00 -> 62.2 mm
- net +5V: track 734.0 -> 744.0 mm
- net /d4: track 160.7 -> 151.9 mm
- net /d2: track 187.0 -> 179.2 mm
- net /d8: track 106.8 -> 99.0 mm
- net /d7: track 107.0 -> 112.3 mm
- net /d6: track 127.2 -> 122.3 mm
- net /d5: track 146.0 -> 143.4 mm
- net /d3: track 173.8 -> 172.8 mm
- net GND: vias 0 -> 2
Other:
- outline, holes or cut-outs redrawn

Commit message: Add SPI and SYNC pins
Connections:
- J1 pad 18: unconnected-(J1-Pin_18-Pad18) -> /SYNC
- J1 pad 19: unconnected-(J1-Pin_19-Pad19) -> /SPI_MOSI
- J1 pad 21: unconnected-(J1-Pin_21-Pad21) -> /SPI_MISO
- J1 pad 23: unconnected-(J1-Pin_23-Pad23) -> /SPI_CLK
- XA1 pad 5V1: unconnected-(XA1-5V-Pad5V1) -> +5V
- XA1 pad D50: unconnected-(XA1-PadD50) -> /SPI_MISO
- XA1 pad D51: unconnected-(XA1-PadD51) -> /SPI_MOSI
- XA1 pad D52: unconnected-(XA1-PadD52) -> /SPI_CLK
- XA1 pad D53: unconnected-(XA1-D53_SS-PadD53) -> +5V
- XA1 pad GND1: unconnected-(XA1-GND-PadGND1) -> GND
Routing:
- net +5V: track 744.0 -> 884.4 mm
- net (no net): track 2.41 -> 0.00 mm

Commit message: Some progress with the peer
Connections:
- XA1 pad D47: unconnected-(XA1-PadD47) -> /SYNC
Routing:
- net /SPI_MISO: track 0.00 -> 100.8 mm, vias 0 -> 1
- net /SPI_CLK: track 0.00 -> 97.2 mm, vias 0 -> 1
- net /SYNC: track 0.00 -> 96.5 mm
- net /SPI_MOSI: track 0.00 -> 87.5 mm
- net /dB: track 59.2 -> 60.5 mm
- net +5V: track 884.4 -> 883.8 mm
- net GND: vias 2 -> 17
